Commit message: Arena for Robocon 24?

File: spark_description/urdf/spark_description.xacro (robot description, xacro)
@@ -270,15 +270,24 @@
     <parent link="front_lidar_base" />
     <child link="front_lidar_sensor" />
+    <!-- Actual -->
     <origin xyz="0.035 0 0.045" rpy="0 0 0" />
+    <!-- For Robocon  -->
+    <!-- <origin xyz="0.145 0 -0.045" rpy="0 0 0" /> -->
   </joint>
   <joint name="rear_lidar_sensor_joint" type="fixed">
     <parent link="rear_lidar_base" />
     <child link="rear_lidar_sensor" />
+    <!-- Actual -->
     <origin xyz="0.035 0 0.045" rpy="0 0 0" />
+    <!-- For Robocon  -->
+    <!-- <origin xyz="-0.075 0 -0.045" rpy="0 0 0" /> -->
   </joint>
   <joint name="merger_lidar_joint" type="fixed">
     <parent link="base_link" />
     <child link="merge_lidar" />
+    <!-- Actual -->
     <origin xyz="0.0 0.0 0.161" rpy="0 0 0" />
+    <!-- For Robocon  -->
+    <!-- <origin xyz="0.0 0.0 0.05" rpy="0 0 0" /> -->
   </joint>
   <joint name="imu_joint" type="fixed">

Commit message: Got R2 working

File: spark_description/urdf/spark_description.xacro (robot description, xacro)
@@ -270,16 +270,10 @@
     <parent link="front_lidar_base" />
     <child link="front_lidar_sensor" />
-    <!-- Actual -->
     <origin xyz="0.035 0 0.045" rpy="0 0 0" />
-    <!-- For Robocon  -->
-    <!-- <origin xyz="0.145 0 -0.045" rpy="0 0 0" /> -->
   </joint>
   <joint name="rear_lidar_sensor_joint" type="fixed">
     <parent link="rear_lidar_base" />
     <child link="rear_lidar_sensor" />
-    <!-- Actual -->
     <origin xyz="0.035 0 0.045" rpy="0 0 0" />
-    <!-- For Robocon  -->
-    <!-- <origin xyz="-0.075 0 -0.045" rpy="0 0 0" /> -->
   </joint>
   <joint name="merger_lidar_joint" type="fixed">
@@ -288,6 +282,4 @@
     <!-- Actual -->
     <origin xyz="0.0 0.0 0.161" rpy="0 0 0" />
-    <!-- For Robocon  -->
-    <!-- <origin xyz="0.0 0.0 0.05" rpy="0 0 0" /> -->
   </joint>
   <joint name="imu_joint" type="fixed">

Commit message: Using house for Spark

File: spark_description/urdf/spark_description.xacro (robot description, xacro)
@@ -16,4 +16,6 @@
         <mesh filename="file://$(find spark_description)/meshes/base_link.stl"
           scale="0.001 0.001 0.001" />
+        <!-- <mesh filename="file://$(find spark_description)/meshes/base_link.stl"
+          scale="0.001 0.001 0.0005" /> -->
       </geometry>
       <material name="cyan" />
@@ -24,4 +26,6 @@
         <mesh filename="file://$(find spark_description)/meshes/base_link.stl"
           scale="0.001 0.001 0.001" />
+        <!-- <mesh filename="file://$(find spark_description)/meshes/base_link.stl"
+          scale="0.001 0.001 0.0005" /> -->
       </geometry>
     </collision>
@@ -271,4 +275,5 @@
     <child link="front_lidar_sensor" />
     <origin xyz="0.035 0 0.045" rpy="0 0 0" />
+    <!-- <origin xyz="0.035 0 -0.035" rpy="0 0 0" /> -->
   </joint>
   <joint name="rear_lidar_sensor_joint" type="fixed">
@@ -276,10 +281,11 @@
     <child link="rear_lidar_sensor" />
     <origin xyz="0.035 0 0.045" rpy="0 0 0" />
+    <!-- <origin xyz="0.035 0 -0.035" rpy="0 0 0" /> -->
   </joint>
   <joint name="merger_lidar_joint" type="fixed">
     <parent link="base_link" />
     <child link="merge_lidar" />
-    <!-- Actual -->
     <origin xyz="0.0 0.0 0.161" rpy="0 0 0" />
+    <!-- <origin xyz="0.0 0.0 0.051" rpy="0 0 0" /> -->
   </joint>
   <joint name="imu_joint" type="fixed">

Commit message: Push for long term no dev

File: spark_description/urdf/spark_description.xacro (robot description, xacro)
@@ -210,23 +210,23 @@
   </link>
   <link name="imu_link">
-		<inertial>
-			<origin rpy="0 0 0" xyz="-0.005006317892412869 0.010331821776814253 0.0005641458401822869"/>
-			<mass value="0.0005786974233911084"/>
-			<inertia ixx="0.0" ixy="0.0" ixz="-0.0" iyy="0.0" iyz="-0.0" izz="0.0"/>
-		</inertial>
-		<visual>
-			<origin rpy="0 0 0" xyz="-0.04 0.01025 -0.10543"/>
-			<geometry>
-				<mesh filename="file://$(find spark_description)/meshes/imu.stl" scale="0.001 0.001 0.001"/>
-			</geometry>
-			<material name="white"/>
-		</visual>
-		<collision>
-			<origin rpy="0 0 0" xyz="-0.04 0.01025 -0.10543"/>
-			<geometry>
-				<mesh filename="file://$(find spark_description)/meshes/imu.stl" scale="0.001 0.001 0.001"/>
-			</geometry>
-		</collision>
-	</link>
+    <inertial>
+      <origin rpy="0 0 0" xyz="-0.005006317892412869 0.010331821776814253 0.0005641458401822869" />
+      <mass value="0.0005786974233911084" />
+      <inertia ixx="0.0" ixy="0.0" ixz="-0.0" iyy="0.0" iyz="-0.0" izz="0.0" />
+    </inertial>
+    <visual>
+      <origin rpy="0 0 0" xyz="-0.04 0.01025 -0.10543" />
+      <geometry>
+        <mesh filename="file://$(find spark_description)/meshes/imu.stl" scale="0.001 0.001 0.001" />
+      </geometry>
+      <material name="white" />
+    </visual>
+    <collision>
+      <origin rpy="0 0 0" xyz="-0.04 0.01025 -0.10543" />
+      <geometry>
+        <mesh filename="file://$(find spark_description)/meshes/imu.stl" scale="0.001 0.001 0.001" />
+      </geometry>
+    </collision>
+  </link>
   <joint name="left_wheel_joint" type="continuous">
     <origin xyz="0.0 0.15 0.04" rpy="0 0 0" />
@@ -294,3 +294,48 @@
     <origin xyz="0.0 0.0 0.05" rpy="0 0 0" />
   </joint>
+  <!-- ################################## ARM ################################## -->
+  <!-- import main macro -->
+  <xacro:include filename="$(find spark_description)/urdf/inc/ur_macro.xacro" />
+  <!-- parameters -->
+  <xacro:arg name="joint_limit_params"
+    default="$(find spark_description)/config/ur3/joint_limits.yaml" />
+  <xacro:arg name="kinematics_params"
+    default="$(find spark_description)/config/ur3/default_kinematics.yaml" />
+  <xacro:arg name="physical_params"
+    default="$(find spark_description)/config/ur3/physical_parameters.yaml" />
+  <xacro:arg name="visual_params"
+    default="$(find spark_description)/config/ur3/visual_parameters.yaml" />
+  <!-- legal values:
+           - hardware_interface/PositionJointInterface
+           - hardware_interface/VelocityJointInterface
+           - hardware_interface/EffortJointInterface
+     -->
+  <!--common
+  parameters -->
+  <xacro:arg name="transmission_hw_interface" default="hardware_interface/PositionJointInterface" />
+  <xacro:arg name="safety_limits" default="false" />
+  <xacro:arg name="safety_pos_margin" default="0.15" />
+  <xacro:arg name="safety_k_position" default="20" />
+  <!-- arm -->
+  <xacro:ur_robot
+    prefix=""
+    joint_limits_parameters_file="$(arg joint_limit_params)"
+    kinematics_parameters_file="$(arg kinematics_params)"
+    physical_parameters_file="$(arg physical_params)"
+    visual_parameters_file="$(arg visual_params)"
+    transmission_hw_interface="$(arg transmission_hw_interface)"
+    safety_limits="$(arg safety_limits)"
+    safety_pos_margin="$(arg safety_pos_margin)"
+    safety_k_position="$(arg safety_k_position)" />
+  <joint name="amr_to_robot" type="fixed">
+    <parent link="base_link" />
+    <child link="ur_base_link" />
+    <origin xyz="0.0 0.0 0.115" rpy="0 0 0" />
+  </joint>
+  <link name="tool0_controller" />
+  <joint name="tool_controller_fake_joint" type="fixed">
+    <parent link="tool0" />
+    <child link="tool0_controller" />
+    <origin xyz="0 0 0" rpy="0 0 0" />
+  </joint>
 </robot>
